Commit message: update by Google AI Studio

File: arm.urdf (robot description, URDF)
Before this commit: robot simple_arm, 4 links, 3 joints
Links:
- link base_link: mass None -> 1.0; geometry collision cylinder length=0.1 radius=0.1; visual cylinder length=0.1 radius=0.1
- link link1: mass None -> 1.0; geometry collision cylinder length=0.5 radius=0.04; visual cylinder length=0.5 radius=0.04
- link link2: mass None -> 0.8; geometry collision cylinder length=0.4 radius=0.03; visual cylinder length=0.4 radius=0.03
- link link3: mass None -> 0.5; geometry collision cylinder length=0.2 radius=0.02; visual cylinder length=0.2 radius=0.02
